File: lamoka1hardware/boostconverter/boostconverter.kicad_pcb (KiCad board)
At the start: 2 copper layers, 11 parts

Commit message: ADD alot of work (I dont even remember what i did lol)
Parts:
- added C2: UUX2A470MNL1GS, footprint:PCAP_10x10-ELECT_NCA, F.Cu at (148.5, 133.0)
- added C3: UUX2A470MNL1GS, footprint:PCAP_10x10-ELECT_NCA, F.Cu at (170.0, 131.5)
- added C4: UCD2A220MNL1GS, incapsmall:PCAP_8x10-ELECT_NCH, F.Cu at (148.5, 122.0)
- added C5: KRM55WR72A226MH01L, KRM55WR72A226MH01L-kicadfiles:CAPC6153X670N, F.Cu at (158.5, 128.5)
- added C6: UCD2A101MNJ1MS, footprint3:CAP_UCD2A_NCH, F.Cu at (187.0, 117.5)
- added IC1: SDM1U100S1F-7, SDM1U100S1F-7-kicadfiles:SODFL3518X115N, F.Cu at (182.7, 130.6)
- added IC2: SDM1U100S1F-7, SDM1U100S1F-7-kicadfiles:SODFL3518X115N, F.Cu at (182.7, 133.9)
- moved SLAVE1 8.70 mm to (160.5, 120.5)
- moved MASTER1 7.16 mm to (170.5, 121.0)
