File: HARDWARE/kicadfiles/Lamoka1/Boost.kicad_sch (KiCad schematic)
At the start: 43 parts, among them Q1 CSD19531Q5A, Q2 CSD19531Q5A, Q3 CSD19531Q5A, Q4 CSD19531Q5A, Q5 AO3400A, U2 LM5122QMHE/NOPB, U3 LM5122QMHE/NOPB

Commit message: Improving everything for boost converter section
Parts:
- removed R41: 47k, symbol Device:R
- added NT1, NT2, NT3, NT4: NetTie_2, NetTie:NetTie-2_SMD_Pad0.5mm, symbol Device:NetTie_2
- added R6: 47k, Components:RC0805N_YAG, symbol 2026-07-01_14-01-11:RC0805FR-0747KL
Connections:
- net FBS: now also NT2.1; no longer C5.2, D8.2 (A), U3.17 (VCC)
- net MODE: now also R6.2
- net SYNCIN/RTS: now also NT3.1; no longer U2.1 (SYNCOUT)
- net VCCM: now also R6.1
- net VIN-SOURCE: now also NT4.1; no longer C25.1, C26.1, C27.1, R39.1, R40.1, R5.2, U2.4 (CSP), U2.5 (VIN), U3.4 (CSP), U3.5 (VIN)
- net Earth renamed GNDPWR
- net GNDPWR: now also NT1.2; no longer C1.1, C29.1, Q5.2 (S), R2.1, R36.2, R38.1, R4.1, R42.2, TP4.1, TP5.1, U2.2 (OPT), U2.9 (AGND), U3.2 (OPT), U3.9 (AGND)
- new net CSPM: C25.1, C26.1, C27.1, NT4.2, R39.1, R40.1, R5.2, U2.4 (CSP), U2.5 (VIN), U3.4 (CSP), U3.5 (VIN)
- new net GNDA: C1.1, C29.1, NT1.1, Q5.2 (S), R2.1, R36.2, R38.1, R4.1, R42.2, TP4.1, TP5.1, U2.2 (OPT), U2.9 (AGND), U3.2 (OPT), U3.9 (AGND)
- new net SYNCOUT: NT3.2, U2.1 (SYNCOUT)
- new net VCCS: C5.2, D8.2 (A), NT2.2, U3.17 (VCC)
Other:
- note added: "Sets restart time for converter"
- note removed: "Sets restart time for converter to around 56ms"
- moved on the sheet: C2, R1, R38, R42, U2, U3

Commit message: Working on getting the PCB layout setup for the boost converter
Parts:
- added J1: Boostconverteroutput, Connector_Wire:SolderWire-0.1sqmm_1x01_D0.4mm_OD1mm, symbol Connector:Conn_01x01_Pin
- added J2: Boostconverterinput, Connector_Wire:SolderWire-0.1sqmm_1x01_D0.4mm_OD1mm, symbol Connector:Conn_01x01_Pin
- added J3: Groundconnection, Connector_Wire:SolderWire-0.1sqmm_1x01_D0.4mm_OD1mm, symbol Connector:Conn_01x01_Pin
Connections:
- net CSPM: now also J2.1 (Pin_1)
- net GNDA: now also J3.1 (Pin_1)
- net VOUT-BOOST: now also J1.1 (Pin_1)
Other:
- moved on the sheet: NT1, NT2
