File: HARDWARE/kicadfiles/Lamoka1/Lamoka1.kicad_pcb (KiCad board)
At the start: 2 copper layers, 42 parts, among them Q1 CSD19531Q5A, Q2 CSD19531Q5A, Q3 CSD19531Q5A, Q4 CSD19531Q5A, Q5 AO3400A, U2 LM5122QMHE/NOPB, U3 LM5122QMHE/NOPB

Commit message: Improving everything for boost converter section
Parts:
- added NT1: NetTie_2, NetTie:NetTie-2_SMD_Pad0.5mm, F.Cu at (145.8, 128.6)
- added NT2: NetTie_2, NetTie:NetTie-2_SMD_Pad0.5mm, F.Cu at (145.8, 130.1)
- added NT3: NetTie_2, NetTie:NetTie-2_SMD_Pad0.5mm, F.Cu at (145.8, 131.6)
- added NT4: NetTie_2, NetTie:NetTie-2_SMD_Pad0.5mm, F.Cu at (145.8, 133.1)
- added R6: 47k, Components:RC0805N_YAG, F.Cu at (154.0, 132.9)
- moved C29 17.8 mm to (166.7, 126.8)
- moved R2 6.02 mm to (162.7, 126.8)
- moved C2 5.72 mm to (158.2, 132.7)
- moved R5 5.50 mm to (162.6, 129.3)
- moved C27 3.04 mm to (132.2, 129.1)
- moved R38 3.04 mm to (149.8, 128.8)
- moved C1 3.04 mm to (181.7, 112.3)
- moved C25 3.04 mm to (132.2, 104.8)
- moved C26 3.04 mm to (132.2, 116.9)
- moved C3 3.04 mm to (181.4, 100.3)
- moved C33 3.04 mm to (156.0, 121.1)
- moved C36 3.04 mm to (150.2, 108.2)
- moved C4 3.04 mm to (155.4, 126.3)
- moved C5 3.04 mm to (181.4, 103.6)
- moved C6 3.04 mm to (155.4, 129.7)
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Connections:
- C1 pad 1: Earth -> GNDA
- C25 pad 2: Earth -> GNDPWR
- C26 pad 2: Earth -> GNDPWR
- C27 pad 2: Earth -> GNDPWR
- C29 pad 1: Earth -> GNDA
- C3 pad 1: Earth -> GNDPWR
- C33 pad 1: Earth -> GNDPWR
- C35 pad 2: Earth -> GNDPWR
- C36 pad 2: Earth -> GNDPWR
- C5 pad 1: Earth -> GNDPWR
- C5 pad 2: /BOOST-SECTION/FBS -> /BOOST-SECTION/VCCS
- D8 pad 2: /BOOST-SECTION/FBS -> /BOOST-SECTION/VCCS
- Q1 pad 1: Earth -> GNDPWR
- Q1 pad 2: Earth -> GNDPWR
- Q1 pad 3: Earth -> GNDPWR
- Q3 pad 1: Earth -> GNDPWR
- Q3 pad 2: Earth -> GNDPWR
- Q3 pad 3: Earth -> GNDPWR
- Q5 pad 2: Earth -> GNDA
- R2 pad 1: Earth -> GNDA
- R36 pad 2: Earth -> GNDA
- R38 pad 1: Earth -> GNDA
- R4 pad 1: Earth -> GNDA
- R42 pad 2: Earth -> GNDA
- TP3 pad 1: Earth -> GNDPWR
- TP4 pad 1: Earth -> GNDA
- TP5 pad 1: Earth -> GNDA
- TP6 pad 1: Earth -> GNDPWR
- TP7 pad 1: Earth -> GNDPWR
- TP8 pad 1: Earth -> GNDPWR
- U2 pad 1: /BOOST-SECTION/SYNCIN/RTS -> /BOOST-SECTION/SYNCOUT
- U2 pad 15: Earth -> GNDPWR
- U2 pad 2: Earth -> GNDA
- U2 pad 9: Earth -> GNDA
- U3 pad 15: Earth -> GNDPWR
- U3 pad 17: /BOOST-SECTION/FBS -> /BOOST-SECTION/VCCS
- U3 pad 2: Earth -> GNDA
- U3 pad 9: Earth -> GNDA

Commit message: Working on getting the PCB layout setup for the boost converter
Parts:
- removed Q5: AO3400A, Components:SOT-23-3L_AOS
- removed R6: 47k, Components:RC0805N_YAG
- added J1: Boostconverteroutput, Connector_Wire:SolderWire-0.1sqmm_1x01_D0.4mm_OD1mm, F.Cu at (264.0, 93.0)
- added J2: Boostconverterinput, Connector_Wire:SolderWire-0.1sqmm_1x01_D0.4mm_OD1mm, F.Cu at (95.7, 57.5)
- added J3: Groundconnection, Connector_Wire:SolderWire-0.1sqmm_1x01_D0.4mm_OD1mm, F.Cu at (236.3, 60.6)
- moved TP6 175.9 mm to (38.0, 17.0)
- moved TP1 163.9 mm to (23.0, 47.5)
- moved TP7 161.9 mm to (24.8, 152.0)
- moved Q1 146.7 mm to (45.2, 17.1)
- moved Q2 146.7 mm to (45.2, 23.9)
- moved Q3 139.3 mm to (32.5, 159.1)
- moved Q4 139.3 mm to (32.5, 165.8)
- moved TP2 137.5 mm to (33.5, 126.5)
- moved R39 135.4 mm to (35.5, 38.5), turned to -90 degrees
- moved R3 130.9 mm to (277.7, 93.5)
- moved R4 130.9 mm to (277.7, 96.0)
- moved L8 126.0 mm to (54.8, 131.5)
- moved R38 123.1 mm to (272.8, 122.0)
- moved C36 122.4 mm to (266.8, 71.1)
- moved C35 116.0 mm to (265.3, 55.1)
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
Commit message: Reconfiguring the BOM, other misc tasks
Parts:
- C27: footprint Components:PCAP_10x10-ELECT_NCA -> Components:PCAP_8x10-ELECT_NCH
- C36: footprint Components:CAP_UCD2A_NCH -> Components:PCAP_8x10-ELECT_NCH
- moved TP6 160.0 mm to (158.2, 122.7)
- moved C35 158.2 mm to (118.7, 114.5)
- moved C36 157.5 mm to (118.7, 124.6)
- moved TP1 145.6 mm to (150.1, 118.6)
- moved R39 141.7 mm to (162.3, 101.8), turned to 0 degrees
- moved TP7 141.4 mm to (162.2, 118.6)
- moved C6 125.0 mm to (136.5, 128.7)
- moved C4 124.1 mm to (136.5, 125.2)
- moved R40 122.9 mm to (162.3, 106.9), turned to 0 degrees
- moved U3 120.1 mm to (153.0, 112.2)
- moved Q1 119.5 mm to (128.8, 102.6)
- moved Q2 119.5 mm to (128.8, 109.3)
- moved TP5 118.0 mm to (158.2, 118.6)
- moved TP2 116.6 mm to (150.1, 122.7)
- moved R3 114.7 mm to (166.2, 120.3)
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