File: HARDWARE/kicadfiles/Lamoka1/Control-section.kicad_sch (KiCad schematic)
At the start: 50 parts, among them J3 USB_C_Receptacle_USB2.0_14P, SW1 PTS636 SM43J SMTR LFS, U1 RP2354A, U2 AMS1117-3.3, U3 74AHCT1G125, X1 ABM8-272-T3

Commit message: Moving everything to the correct locations
Parts:
- U1: Manufacturer Raspberry Pi -> Raspberry Pi
Changed lines of the file:
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@@
 			)
 		)
-		(property "Manufacturer" "Raspberry Pi"
+		(property "Manufacturer" "	\nRaspberry Pi"
 			(at 196.85 100.33 0)
 			(hide yes)

Commit message: Finishing routing for H bridge (Inversion-section)
Connections:
- net GPIO1: now reaches U1.3 (GPIO1)
- net GPIO2: now reaches U1.4 (GPIO2)
- net GPIO3: now reaches U1.5 (GPIO3)
- net GPIO4: now reaches U1.7 (GPIO4)
Other:
- moved on the sheet: C1, C10, C11, C2, C3, C4, C5, C6, C7, C8, C9, D1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

Commit message: ADD logo, repo grade, and cosmetic/finishing H bridge connections
Connections:
- net GPIO11: no longer U3.2
- no-connect marks 26 -> 32
Changed lines of the file:
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@@
+	)
+	(no_connect
+		(at 222.25 77.47)
 	)
 	(no_connect
@@
 	)
 	(no_connect
+		(at 222.25 87.63)
+	)
+	(no_connect
 		(at 222.25 123.19)
 	)
@@
 	)
 	(no_connect
+		(at 222.25 74.93)
+	)
+	(no_connect
 		(at 222.25 125.73)
 	)
@@
 	)
 	(no_connect
+		(at 222.25 85.09)
+	)
+	(no_connect
 		(at 222.25 113.03)
 	)
 	(no_connect
+		(at 222.25 80.01)
+	)
+	(no_connect
 		(at 222.25 105.41)
 	)
@@
 	(no_connect
 		(at 222.25 135.89)
+	)
+	(no_connect
+		(at 222.25 82.55)
 	)
 	(no_connect
@@
 		)
 	)
-	(label "GPIO4"
-		(at 222.25 72.39 0)
-		(effects
-			(font
-				(size 1.27 1.27)
-			)
-			(justify left bottom)
-		)
-	)
-	(label "GPIO1"
-		(at 222.25 64.77 0)
-		(effects
-			(font
-				(size 1.27 1.27)
-			)
-			(justify left bottom)
-		)
-	)
 	(label "BTN"
 		(at 229.87 62.23 0)
@@
 		)
 	)
-	(label "GPIO3"
-		(at 222.25 69.85 0)
+	(label "GPIO11"
+		(at 222.25 90.17 0)
 		(effects
 			(font
@@
 		)
 	)
-	(label "GPIO2"
-		(at 222.25 67.31 0)
-		(effects
-			(font
-				(size 1.27 1.27)
-			)
-			(justify left bottom)
-		)
-	)
 	(label "USB_DP"
 		(at 134.62 62.23 0)
@@
 		)
 	)
+	(label "GPIO11"
+		(at 53.34 176.53 90)
+		(effects
+			(font
+				(size 1.27 1.27)
+			)
+			(justify left bottom)
+		)
+	)
 	(label "5V"
 		(at 137.16 245.11 180)
@@
 		)
 	)
-	(hierarchical_label "GPIO11"
+	(hierarchical_label "GPIO1"
 		(shape input)
-		(at 222.25 90.17 0)
+		(at 222.25 64.77 0)
 		(effects
 			(font
@@
 		)
 	)
-	(hierarchical_label "GPIO11"
+	(hierarchical_label "GPIO3"
 		(shape input)
-		(at 50.8 181.61 180)
-		(effects
-			(font
-				(size 1.27 1.27)
-			)
-			(justify right)
-		)
-	)
+		(at 222.25 69.85 0)
+		(effects
+			(font
+				(size 1.27 1.27)
+			)
+			(justify left)
+		)
+	)
+	(hierarchical_label "GPIO4"
+		(shape input)
+		(at 222.25 72.39 0)
+		(effects
+			(font
+				(size 1.27 1.27)
+			)
+			(justify left)
+		)
+	)
+	(hierarchical_label "GPIO2"
+		(shape input)
+		(at 222.25 67.31 0)
+		(effects
+			(font
+				(size 1.27 1.27)
+			)
+			(justify left)
+		)
+	)

Commit message: Improving repository
Other:
- title: Controling  -> Control-Section
- moved on the sheet: C14, C17, R2, R3, R5, R6

Commit message: ADD fan connection, and finish buck converter 5v
Parts:
- added C24: TMK212BBJ106KG, CAP_TMK212_TAY, symbol TMK212BBJ106KG:TMK212BBJ106KG
- added C25: GRM31CR71A226KE15L, G-31_MUR, symbol GRM31CR71A226KE15L:GRM31CR71A226KE15L
- added CR1, CR2: SS14-E3/61T, DO-214AC_VIS, symbol SS14-E3/61T:SS14-E3_61T
- added J4: 470531000, CONN_SD-47053-001_H10p00_MOL, symbol 470531000:470531000
- added L3: PA4332.222NLT, IND_PA4332.222NLT_PUL, symbol PA4332.222NLT:PA4332.222NLT
- added R19: RC0603FR-07180KL, RC0603N_YAG, symbol RC0603FR-07180KL:RC0603FR-07180KL
- added R20: CRCW0402953KFKED, RC0402N_VIS, symbol CRCW0402953KFKED:CRCW0402953KFKED
- added R21: CRCW0402100KFKED, RES_CRCW_0402_VIS, symbol CRCW0402100KFKED:CRCW0402100KFKED
- added U7: TPS62160DSGR, DSG8_1P6X0P9, symbol TPS62160DSGR:TPS62160DSGR
Connections:
- net 5V: now also CR1.1, CR2.1; no longer J3.A4 (VBUS), J3.A9 (VBUS), J3.B4 (VBUS), J3.B9 (VBUS)
- net GND: now also C24.2, C25.1, J4.1, R19.2, U7.1 (PGND), U7.4 (AGND), U7.9 (EPAD)
- net GPIO5: now reaches U1.8 (GPIO5)
- net GPIO5: now also J4.3
- net GPIO6: now reaches U1.9 (GPIO6)
- net GPIO6: now also J4.4
- new net: R19.1, R20.2, U7.5 (FB)
- new net: L3.2, U7.7 (SW)
- new net 11-14v input: C24.1, U7.2 (VIN), U7.3 (EN)
- new net Buck-5v: C25.2, CR2.2, J4.2, L3.1, R20.1, R21.1, U7.6 (VOS)
- new net PG: R21.2, U7.8 (PG)
- new net USB-5v: CR1.2, J3.A4 (VBUS), J3.A9 (VBUS), J3.B4 (VBUS), J3.B9 (VBUS)
- no-connect marks 32 -> 30
Other:
- note added: "11-14v to 5v"
- note added: "Buck-Sub-Section"
- note added: "Diode-Power OR-ing"
- note added: "Fan-connection"
- moved on the sheet: C12

Commit message: ADD temp sensors, more doccumentation regarding design
Parts:
- added R22: 10k, DBZ0003A-IPC_A, symbol Device:R
- added U8: TMP235A2DBZR, DBZ0003A-IPC_A, symbol TMP235A2DBZR:TMP235A2DBZR
Connections:
- net GND: now also U8.3 (GND)
- net GPIO11: now also U3.2
- net GPIO5: now also R22.2
- net TEMP_CTRL: now reaches U1.10 (GPIO7)
- net TEMP_CTRL: now also U8.2 (VOUT)
- net TEMP_INV: now reaches U1.12 (GPIO8)
- net 3V3 renamed 3v3
- net 3v3: now also R22.1, U8.1 (VDD)
- no-connect marks 30 -> 28
Other:
- note added: "Temperature-Sensor"

Commit message: Giving Q1 and Q2 values that represent their respected MPNs. Changing temp sensor outputs to ADC pins instead of regular GPIO. Correcting design notes to reflect new GPIO pin change
Connections:
- net TEMP_CTRL: now also U1.40 (GPIO26/ADC0); no longer U1.10 (GPIO7)
- net TEMP_INV: now also U1.41 (GPIO27/ADC1); no longer U1.12 (GPIO8)
Changed lines of the file:
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@@
+	)
+	(no_connect
+		(at 222.25 80.01)
 	)
 	(no_connect
@@
 	)
 	(no_connect
-		(at 222.25 133.35)
-	)
-	(no_connect
 		(at 171.45 133.35)
 	)
@@
 	)
 	(no_connect
+		(at 222.25 82.55)
+	)
+	(no_connect
 		(at 222.25 125.73)
 	)
@@
 	(no_connect
 		(at 222.25 97.79)
-	)
-	(no_connect
-		(at 222.25 130.81)
 	)
 	(no_connect
@@
 		)
 	)
-	(label "TEMP_CTRL"
-		(at 222.25 80.01 0)
-		(effects
-			(font
-				(size 1.27 1.27)
-			)
-			(justify left bottom)
-		)
-	)
 	(label "GPIO5"
 		(at 229.87 74.93 0)
@@
 		)
 	)
+	(label "TEMP_CTRL"
+		(at 222.25 130.81 0)
+		(effects
+			(font
+				(size 1.27 1.27)
+			)
+			(justify left bottom)
+		)
+	)
 	(label "1V1"
 		(at 214.63 46.99 0)
@@
 			)
 			(justify right bottom)
-		)
-	)
-	(hierarchical_label "TEMP_INV"
-		(shape input)
-		(at 222.25 82.55 0)
-		(effects
-			(font
-				(size 1.27 1.27)
-			)
-			(justify left)
 		)
 	)
@@
 		(effects
 			(font
+				(size 1.27 1.27)
+			)
+			(justify left)
+		)
+	)
+	(hierarchical_label "TEMP_INV"
+		(shape input)
+		(at 222.25 133.35 0)
+		(effects
+			(font

Commit message: ADD better format for connectors, output connector, transformer connector, and more
Parts:
- removed J3: USB_C_Receptacle_USB2.0_14P, Connector_USB:USB_C_Receptacle_HRO_TYPE-C-31-M-12, symbol Connector:USB_C_Receptacle_USB2.0_14P
- removed J4: 470531000, CONN_SD-47053-001_H10p00_MOL, symbol 470531000:470531000
- removed NT2: USB_SHIELD_BOND, symbol Device:NetTie_2
Connections:
- net CC1: now reaches R2.1
- net D+: now reaches R6.1
- net CC2: now reaches R3.1
- net D-: now reaches R5.1
- net USB-5v renamed VBUS
Other:
- note removed: "Fan-connection"
- moved on the sheet: C12, U8
