File: HARDWARE/kicadfiles/Lamoka1/Lamoka1.kicad_sch (KiCad schematic)
At the start: 5 parts, among them J1 2606-1108/010-000, J2 2606-1352, J3 USB_C_Receptacle_USB2.0_14P, J4 470531000, J5 2604-1103

Commit message: MPN fixes, footprint fixes, ADD MUX and voltage sensing. ADD photo in main readme
Parts:
- J1: footprint CONN8_2606-1108/010-000_WAG -> 2606-1108/010-000:CONN8_2606-1108&slash_010-000_WAG
- J2: footprint CONN2_2606-1352_WAG -> 2606-1352:CONN2_2606-1352_WAG
- J4: footprint CONN_SD-47053-001_H10p00_MOL -> 470531000:CONN_SD-47053-001_H10p00_MOL
- J5: footprint CONN3_2604-1103_WAG -> 2604-1103:CONN3_2604-1103_WAG
Other:
- sheet Inversion-Section ports: added 17v; removed none
Changed lines of the file:
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@@
 	(title_block
 		(company "Flamingo & Cactus")
+		(comment 1 "Please do not consider this as a finished schematic, change is constant.")
+		(comment 2 "License: CERN-OHL-W-2.0")
+		(comment 3 "https://github.com/bearjhartjen/Lamoka1-project")
 	)
 	(rectangle
@@
 			)
 		)
-		(property "Footprint" "CONN2_2606-1352_WAG"
+		(property "Footprint" "2606-1352:CONN2_2606-1352_WAG"
 			(at 152.4 43.18 0)
 			(hide yes)
@@
 		)
 		(property "Description" ""
+			(at 152.4 43.18 0)
+			(hide yes)
+			(show_name no)
+			(do_not_autoplace no)
+			(effects
+				(font
+					(size 1.27 1.27)
+				)
+			)
+		)
+		(property "KLC_S4.2_DVDD" ""
+			(at 152.4 43.18 0)
+			(hide yes)
+			(show_name no)
+			(do_not_autoplace no)
+			(effects
+				(font
+					(size 1.27 1.27)
+				)
+			)
+		)
+		(property "KLC_S4.2_VREG_LX" ""
 			(at 152.4 43.18 0)
 			(hide yes)
@@
 			)
 		)
-		(property "Footprint" "CONN3_2604-1103_WAG"
+		(property "Footprint" "2604-1103:CONN3_2604-1103_WAG"
 			(at 261.62 91.44 0)
 			(hide yes)
@@
 		)
 		(property "Description" ""
+			(at 261.62 91.44 0)
+			(hide yes)
+			(show_name no)
+			(do_not_autoplace no)
+			(effects
+				(font
+					(size 1.27 1.27)
+				)
+			)
+		)
+		(property "KLC_S4.2_DVDD" ""
+			(at 261.62 91.44 0)
+			(hide yes)
+			(show_name no)
+			(do_not_autoplace no)
+			(effects
+				(font
+					(size 1.27 1.27)
+				)
+			)
+		)
+		(property "KLC_S4.2_VREG_LX" ""
 			(at 261.62 91.44 0)
 			(hide yes)
@@
 			)
 		)
-		(property "Footprint" "CONN8_2606-1108/010-000_WAG"
+		(property "Footprint" "2606-1108/010-000:CONN8_2606-1108&slash_010-000_WAG"
 			(at 228.6 54.61 0)
 			(hide yes)
@@
 	(symbol
 		(lib_id "Flamingo&Cactus-logo:LOGO")
-		(at 181.61 173.99 0)
+		(at 279.4 175.26 0)
 		(unit 1)
 		(body_style 1)
@@
 		(fields_autoplaced yes)
 		(property "Reference" "#G1"
-			(at 181.61 169.6241 0)
+			(at 279.4 170.8941 0)
 			(hide yes)
 			(show_name no)
@@
 		)
 		(property "Value" "LOGO"
-			(at 181.61 178.3559 0)
+			(at 279.4 179.6259 0)
 			(hide yes)
 			(show_name no)
@@
 		)
 		(property "Footprint" "Package_LCC:PLCC-84_29.3x29.3mm_P1.27mm"
-			(at 181.61 173.99 0)
+			(at 279.4 175.26 0)
 			(hide yes)
 			(show_name no)
@@
 		)
 		(property "Datasheet" ""
-			(at 181.61 173.99 0)
+			(at 279.4 175.26 0)
 			(hide yes)
 			(show_name no)
@@
 		)
 		(property "Description" ""
-			(at 181.61 173.99 0)
+			(at 279.4 175.26 0)
 			(hide yes)
 			(show_name no)
@@
 			)
 		)
+		(property "MPN" "TYPE-C-31-M-12"
+			(at 29.21 107.95 0)
+			(hide yes)
+			(show_name no)
+			(do_not_autoplace no)
+			(effects
+				(font
+					(size 1.27 1.27)
+				)
+			)
+		)
+		(property "Manufacturer" "HRO Electronics"
+			(at 29.21 107.95 0)
+			(hide yes)
+			(show_name no)
+			(do_not_autoplace no)
+			(effects
+				(font
+					(size 1.27 1.27)
+				)
+			)
+		)
+		(property "Notes" ""
+			(at 29.21 107.95 0)
+			(hide yes)
+			(show_name no)
+			(do_not_autoplace no)
+			(effects
+				(font
+					(size 1.27 1.27)
+				)
+			)
+		)
 		(property "KLC_S4.2_DVDD" ""
 			(at 29.21 107.95 0)
@@
 		)
 		(property "KLC_S4.2_VREG_LX" ""
-			(at 29.21 107.95 0)
-			(hide yes)
-			(show_name no)
-			(do_not_autoplace no)
-			(effects
-				(font
-					(size 1.27 1.27)
-				)
-			)
-		)
-		(property "MPN" "TYPE-C-31-M-12"
-			(at 29.21 107.95 0)
-			(hide yes)
-			(show_name no)
-			(do_not_autoplace no)
-			(effects
-				(font
-					(size 1.27 1.27)
-				)
-			)
-		)
-		(property "Manufacturer" "HRO Electronics"
-			(at 29.21 107.95 0)
-			(hide yes)
-			(show_name no)
-			(do_not_autoplace no)
-			(effects
-				(font
-					(size 1.27 1.27)
-				)
-			)
-		)
-		(property "Notes" ""
-			(at 29.21 107.95 0)
-			(hide yes)
-			(show_name no)
-			(do_not_autoplace no)
-			(effects
-				(font
-					(size 1.27 1.27)
-				)
-			)
-		)
-		(property "Supplier" ""
-			(at 29.21 107.95 0)
-			(hide yes)
-			(show_name no)
-			(do_not_autoplace no)
-			(effects
-				(font
-					(size 1.27 1.27)
-				)
-			)
-		)
-		(property "Supplier Part Number" ""
 			(at 29.21 107.95 0)
 			(hide yes)
@@
 			)
 		)
-		(property "Footprint" "CONN_SD-47053-001_H10p00_MOL"
+		(property "Footprint" "470531000:CONN_SD-47053-001_H10p00_MOL"
 			(at 86.36 64.77 0)
 			(hide yes)
@@
 		)
 		(property "Description" ""
+			(at 86.36 64.77 0)
+			(hide yes)
+			(show_name no)
+			(do_not_autoplace no)
+			(effects
+				(font
+					(size 1.27 1.27)
+				)
+			)
+		)
+		(property "KLC_S4.2_DVDD" ""
+			(at 86.36 64.77 0)
+			(hide yes)
+			(show_name no)
+			(do_not_autoplace no)
+			(effects
+				(font
+					(size 1.27 1.27)
+				)
+			)
+		)
+		(property "KLC_S4.2_VREG_LX" ""
 			(at 86.36 64.77 0)
 			(hide yes)
@@
 			)
 		)
+		(pin "17v" input
+			(at 149.86 120.65 180)
+			(effects
+				(font
+					(size 1.27 1.27)
+				)
+				(justify left)
+			)
+		)

Commit message: ADD source current monitoring, and other features, some more correcting of MPN and footprints
Parts:
- added RCS1: 2m, Resistor_SMD:R_2512_6332Metric, symbol Device:R
Connections:
- net 11-14V input: now also RCS1.1
- new net Control-Section/11-14v input: RCS1.2
Other:
- sheet Control-Section ports: added RCS1-L, RCS1-S; removed none
Changed lines of the file:
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@@
+	)
+	(junction
+		(at 142.24 63.5)
+		(diameter 0)
+		(color 0 0 0 0)
 	)
 	(junction
@@
 	)
 	(junction
-		(at 144.78 93.98)
+		(at 142.24 73.66)
 		(diameter 0)
 		(color 0 0 0 0)
@@
 	)
 	(junction
+		(at 144.78 93.98)
+		(diameter 0)
+		(color 0 0 0 0)
+	)
+	(junction
 		(at 151.13 44.45)
 		(diameter 0)
@@
 	(wire
 		(pts
+			(xy 119.38 63.5) (xy 142.24 63.5)
+		)
+		(stroke
+			(width 0)
+			(type default)
+		)
+	)
+	(wire
+		(pts
 			(xy 228.6 64.77) (xy 217.17 64.77)
 		)
@@
 	(wire
 		(pts
+			(xy 142.24 74.93) (xy 142.24 73.66)
+		)
+		(stroke
+			(width 0)
+			(type default)
+		)
+	)
+	(wire
+		(pts
 			(xy 151.13 49.53) (xy 151.13 50.8)
 		)
@@
 	(wire
 		(pts
-			(xy 144.78 44.45) (xy 144.78 93.98)
-		)
-		(stroke
-			(width 0)
-			(type default)
-		)
-	)
-	(wire
-		(pts
 			(xy 203.2 55.88) (xy 203.2 82.55)
 		)
@@
 	(wire
 		(pts
+			(xy 121.92 82.55) (xy 121.92 73.66)
+		)
+		(stroke
+			(width 0)
+			(type default)
+		)
+	)
+	(wire
+		(pts
 			(xy 50.8 107.95) (xy 44.45 107.95)
 		)
@@
 	(wire
 		(pts
+			(xy 144.78 74.93) (xy 144.78 93.98)
+		)
+		(stroke
+			(width 0)
+			(type default)
+		)
+	)
+	(wire
+		(pts
 			(xy 139.7 113.03) (xy 149.86 113.03)
 		)
@@
 	(wire
 		(pts
+			(xy 144.78 93.98) (xy 149.86 93.98)
+		)
+		(stroke
+			(width 0)
+			(type default)
+		)
+	)
+	(wire
+		(pts
 			(xy 29.21 130.81) (xy 29.21 132.08)
 		)
@@
 	(wire
 		(pts
+			(xy 144.78 44.45) (xy 144.78 62.23)
+		)
+		(stroke
+			(width 0)
+			(type default)
+		)
+	)
+	(wire
+		(pts
 			(xy 228.6 62.23) (xy 217.17 62.23)
 		)
@@
 	(wire
 		(pts
+			(xy 142.24 62.23) (xy 142.24 63.5)
+		)
+		(stroke
+			(width 0)
+			(type default)
+		)
+	)
+	(wire
+		(pts
 			(xy 228.6 69.85) (xy 217.17 69.85)
 		)
@@
 	(wire
 		(pts
+			(xy 144.78 62.23) (xy 142.24 62.23)
+		)
+		(stroke
+			(width 0)
+			(type default)
+		)
+	)
+	(wire
+		(pts
 			(xy 139.7 93.98) (xy 144.78 93.98)
 		)
@@
 	(wire
 		(pts
+			(xy 142.24 73.66) (xy 142.24 72.39)
+		)
+		(stroke
+			(width 0)
+			(type default)
+		)
+	)
+	(wire
+		(pts
 			(xy 50.8 106.68) (xy 64.77 106.68)
 		)
@@
 	(wire
 		(pts
+			(xy 119.38 82.55) (xy 119.38 63.5)
+		)
+		(stroke
+			(width 0)
+			(type default)
+		)
+	)
+	(wire
+		(pts
 			(xy 217.17 55.88) (xy 203.2 55.88)
 		)
@@
 	(wire
 		(pts
-			(xy 144.78 93.98) (xy 149.86 93.98)
-		)
-		(stroke
-			(width 0)
-			(type default)
-		)
-	)
-	(wire
-		(pts
 			(xy 64.77 128.27) (xy 52.07 128.27)
 		)
@@
 	(wire
 		(pts
+			(xy 142.24 74.93) (xy 144.78 74.93)
+		)
+		(stroke
+			(width 0)
+			(type default)
+		)
+	)
+	(wire
+		(pts
 			(xy 261.62 96.52) (xy 255.27 96.52)
 		)
@@
 	(wire
 		(pts
+			(xy 142.24 63.5) (xy 142.24 64.77)
+		)
+		(stroke
+			(width 0)
+			(type default)
+		)
+	)
+	(wire
+		(pts
 			(xy 50.8 123.19) (xy 64.77 123.19)
 		)
@@
 		(pts
 			(xy 231.14 97.79) (xy 255.27 97.79)
+		)
+		(stroke
+			(width 0)
+			(type default)
+		)
+	)
+	(wire
+		(pts
+			(xy 121.92 73.66) (xy 142.24 73.66)
 		)
 		(stroke
@@
 		)
 	)
+	(symbol
+		(lib_id "Device:R")
+		(at 142.24 68.58 0)
+		(unit 1)
+		(body_style 1)
+		(exclude_from_sim no)
+		(in_bom yes)
+		(on_board yes)
+		(in_pos_files yes)
+		(dnp no)
+		(property "Reference" "RCS1"
+			(at 135.636 66.802 0)
+			(show_name no)
+			(do_not_autoplace no)
+			(effects
+				(font
+					(size 1.27 1.27)
+				)
+				(justify left)
+			)
+		)
+		(property "Value" "2m"
+			(at 137.922 68.834 0)
+			(show_name no)
+			(do_not_autoplace no)
+			(effects
+				(font
+					(size 1.27 1.27)
+				)
+				(justify left)
+			)
+		)
+		(property "Footprint" "Resistor_SMD:R_2512_6332Metric"
+			(at 140.462 68.58 90)
+			(hide yes)
+			(show_name no)
+			(do_not_autoplace no)
+			(effects
+				(font
+					(size 1.27 1.27)
+				)
+			)
+		)
+		(property "Datasheet" ""
+			(at 142.24 68.58 0)
+			(hide yes)
+			(show_name no)
+			(do_not_autoplace no)
+			(effects
+				(font
+					(size 1.27 1.27)
+				)
+			)
+		)
+		(property "Description" "Resistor"
+			(at 142.24 68.58 0)
+			(hide yes)
+			(show_name no)
+			(do_not_autoplace no)
+			(effects
+				(font
+					(size 1.27 1.27)
+				)
+			)
+		)
+		(property "MPN" "CSNL2512FT2L00"
+			(at 142.24 68.58 0)
+			(hide yes)
+			(show_name no)
+			(do_not_autoplace no)
+			(effects
+				(font
+					(size 1.27 1.27)
+				)
+			)
+		)
+		(pin "2"
+		)
+		(pin "1"
+		)
+		(instances
+			(project "Lamoka1"
+				(path "/c7bb62b6-932f-49c1-a356-0286e905fc0a"
+					(reference "RCS1")
+					(unit 1)
+				)
+			)
+		)
+	)
 	(sheet
 		(at 149.86 82.55)
@@
 			(effects
 				(font
+					(size 1.27 1.27)
+				)
+				(justify right)
+			)
+		)
+		(pin "RCS1-L" input
+			(at 121.92 82.55 90)
+			(effects
+				(font
+					(size 1.27 1.27)
+				)
+				(justify right)
+			)
+		)
+		(pin "RCS1-S" input
+			(at 119.38 82.55 90)
+			(effects
+				(font
