File: HARDWARE/kicadfiles/Lamoka1/Inversion-section.kicad_sch (KiCad schematic)
At the start: 47 parts, among them J1 Connect to transformer, J2 2606-1352, Q1 NMOS, Q2 NMOS, Q3 CSD19536KCS, Q4 CSD19536KCS, Q5 CSD19536KCS, Q6 CSD19536KCS, U4 LM5122MH/NOPB, U5 UCC27735DR, U6 UCC27735DR, U9 TMP235A2DBZR

Commit message: Giving Q1 and Q2 values that represent their respected MPNs. Changing temp sensor outputs to ADC pins instead of regular GPIO. Correcting design notes to reflect new GPIO pin change
Parts:
- Q1: value NMOS -> CSD16323Q3
- Q2: value NMOS -> CSD17304Q3
Changed lines of the file:
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@@
 		(in_pos_files yes)
 		(dnp no)
-		(fields_autoplaced yes)
 		(property "Reference" "Q2"
 			(at 116.84 48.2599 0)
@@
 			)
 		)
-		(property "Value" "NMOS"
-			(at 116.84 50.7999 0)
+		(property "Value" "CSD17304Q3"
+			(at 115.062 51.054 0)
 			(show_name no)
 			(do_not_autoplace no)
@@
 			)
 		)
-		(property "Value" "NMOS"
+		(property "Value" "CSD16323Q3"
 			(at 119.38 44.45 90)
 			(show_name no)

Commit message: ADD better format for connectors, output connector, transformer connector, and more
Parts:
- removed J1: Connect to transformer, Connector:Tag-Connect_TC2030-IDC-FP_2x03_P1.27mm_Vertical, symbol Connector:Conn_01x02_Pin
- removed J2: 2606-1352, CONN2_2606-1352_WAG, symbol Wago-connector:2606-1352
Connections:
- net GND: now also U4.21 (PAD)
- net G4S renamed SW_B
- net Q3S renamed SW_A
Other:
- note removed: "Wago-connector 2606-1352"

Commit message: MPN fixes, footprint fixes, ADD MUX and voltage sensing. ADD photo in main readme
Parts:
- Cbst1: MPN (none) -> 08053C104KAT2A
- Ccomp1: MPN (none) -> CGA4C2C0G1H392J060AA
- Ccomp2: MPN (none) -> GRM1555C1H131GA01D
- Cin1: MPN (none) -> 20SVPF56MX
- Cout1, Cout2, Cout3: MPN (none) -> 25SVPF180M
- Coutx1: MPN (none) -> C3216X5R1E476M160AC
- Cres1: MPN (none) -> TMK212BJ474KD-T
- Css1: MPN (none) -> GRM155R71A333KA01D
- Cvcc1: MPN (none) -> MSAST21GAB5475MTNAO1
- Cvin1: MPN (none) -> C1005X5R1V474K050BC
- Dbst1: MPN (none) -> SK215ATR
- L2: MPN (none) -> XAL1580-182MEB
- Q1: value CSD16323Q3 -> 25V 60A N-Ch; MPN (none) -> CSD16323Q3
- Q2: value CSD17304Q3 -> 30V 56A N-Ch; MPN (none) -> CSD17304Q3
- Q3, Q4, Q5, Q6: value CSD19536KCS -> 100V 150A N-Ch; MPN (none) -> CSD19536KCS
- Rcomp1: MPN (none) -> RC0201FR-0728K7L
- Rfbb1: MPN (none) -> MPN00CenterCenter00
- Rfbt1, Ruvt1: MPN (none) -> CRCW040249K9FKED
- Rsense1: MPN (none) -> CSNL1206FT2L00
- Rslope1: MPN (none) -> RC0201FR-07105KL
- Rt1: MPN (none) -> CRCW040218K2FKED
- Ruvb1: MPN (none) -> CRCW04027K15FKED
- Rvin1: MPN (none) -> CRCW04023R01FKED
- U4: MPN (none) -> LM5122MH/NOPB
- U5, U6: MPN (none) -> UCC27735DR
- U9: footprint DBZ0003A-IPC_A -> TMP235A2DBZR:DBZ0003A-IPC_A; MPN (none) -> TMP235A2DBZR

Commit message: General work on schem, BOM, footprints. Rout 11-14v to 5v buck converter
Parts:
- R10, R12, U5, U6: footprint SOIC_14L_TEX -> (none)
Changed lines of the file:
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@@
 			)
 		)
-		(property "Footprint" "SOIC_14L_TEX"
+		(property "Footprint" ""
 			(at 265.43 104.14 0)
 			(hide yes)
@@
 			)
 		)
-		(property "Footprint" "SOIC_14L_TEX"
+		(property "Footprint" ""
 			(at 240.03 97.028 90)
 			(hide yes)
@@
 			)
 		)
-		(property "Footprint" "SOIC_14L_TEX"
+		(property "Footprint" ""
 			(at 240.03 108.458 90)
 			(hide yes)
@@
 			)
 		)
-		(property "Footprint" "SOIC_14L_TEX"
+		(property "Footprint" ""
 			(at 265.43 71.12 0)
 			(hide yes)

Commit message: ADD seperate user interface board, improve doccumentation
Parts:
- U4: footprint Components for Lamoka1 general:PWP0020A_N -> LM5122QMHX-NOPB:PWP20_3P0X4P2
Changed lines of the file:
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@@
 			)
 		)
-		(property "Footprint" "Components for Lamoka1 general:PWP0020A_N"
+		(property "Footprint" "LM5122QMHX-NOPB:PWP20_3P0X4P2"
 			(at 55.88 114.3 0)
 			(hide yes)

Commit message: Route whole 11-14v to 17v boost converter
Parts:
- Cbst1: footprint Components for Lamoka1 general:CAPC2012X94N -> Capacitor_SMD:C_0805_2012Metric
- Ccomp1: footprint Components for Lamoka1 general:CAPC2012X75N -> Capacitor_SMD:C_0805_2012Metric
- Ccomp2, Css1, Cvin1: footprint Components for Lamoka1 general:CAPC1005X55N -> Capacitor_SMD:C_0402_1005Metric
- Cin1: footprint Components for Lamoka1 general:CAP_20SVPF56MX -> Capacitor_SMD:CP_Elec_5x5.9
- Cout1, Cout2, Cout3: footprint Components for Lamoka1 general:CAP_25SVPF100M -> Capacitor_SMD:CP_Elec_8x11.9
- Coutx1: footprint Components for Lamoka1 general:CAPC3216X180N -> Capacitor_SMD:C_1206_3216Metric
- Cres1: footprint Components for Lamoka1 general:CAPC2012X95N -> Capacitor_SMD:C_0805_2012Metric
- Cvcc1: footprint Components for Lamoka1 general:CAPC2012X140N -> Capacitor_SMD:C_0805_2012Metric
- Dbst1: footprint (none) -> Diode_SMD:D_SMA
- L2: footprint Components for Lamoka1 general:IND_XAL1580-182MEB -> Inductor_SMD:L_Coilcraft_XAL1580-182
- Q1: footprint (none) -> CSD16323Q3:DQG0008A
- Q2: footprint (none) -> CSD17304Q3:DQG0008A
- Rcomp1, Rslope1: footprint (none) -> Resistor_SMD:R_0201_0603Metric
- Rfbb1: footprint (none) -> Resistor_SMD:R_0402_1005Metric; MPN MPN00CenterCenter00 -> CRCW04023K79FKED
- Rfbt1, Rt1, Ruvb1, Ruvt1, Rvin1: footprint (none) -> Resistor_SMD:R_0402_1005Metric
- Rsense1: footprint (none) -> Resistor_SMD:R_1206_3216Metric
Changed lines of the file:
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@@
 			)
 		)
-		(property "Footprint" ""
+		(property "Footprint" "CSD17304Q3:DQG0008A"
 			(at 115.57 46.99 0)
 			(hide yes)
@@
 			)
 		)
-		(property "Footprint" "Components for Lamoka1 general:CAPC2012X95N"
+		(property "Footprint" "Capacitor_SMD:C_0805_2012Metric"
 			(at 87.3252 74.93 0)
 			(hide yes)
@@
 			)
 		)
-		(property "Footprint" "Components for Lamoka1 general:CAPC1005X55N"
+		(property "Footprint" "Capacitor_SMD:C_0402_1005Metric"
 			(at 149.86 68.8848 0)
 			(hide yes)
@@
 			)
 		)
-		(property "Footprint" "Components for Lamoka1 general:CAPC2012X94N"
+		(property "Footprint" "Capacitor_SMD:C_0805_2012Metric"
 			(at 124.46 84.1248 0)
 			(hide yes)
@@
 			)
 		)
-		(property "Footprint" ""
+		(property "Footprint" "Resistor_SMD:R_0402_1005Metric"
 			(at 62.992 49.53 90)
 			(hide yes)
@@
 			)
 		)
-		(property "Footprint" "Components for Lamoka1 general:CAP_20SVPF56MX"
+		(property "Footprint" "Capacitor_SMD:CP_Elec_5x5.9"
 			(at 54.3052 49.53 0)
 			(hide yes)
@@
 			)
 		)
-		(property "Footprint" "Components for Lamoka1 general:CAPC2012X75N"
+		(property "Footprint" "Capacitor_SMD:C_0805_2012Metric"
 			(at 153.67 80.3148 0)
 			(hide yes)
@@
 			)
 		)
-		(property "Footprint" "Components for Lamoka1 general:CAPC3216X180N"
+		(property "Footprint" "Capacitor_SMD:C_1206_3216Metric"
 			(at 172.4152 45.72 0)
 			(hide yes)
@@
 			)
 		)
-		(property "Footprint" ""
+		(property "Footprint" "Resistor_SMD:R_0402_1005Metric"
 			(at 127.762 58.42 90)
 			(hide yes)
@@
 			)
 		)
-		(property "MPN" "MPN00CenterCenter00"
+		(property "MPN" "CRCW04023K79FKED"
 			(at 129.54 58.42 0)
 			(hide yes)
@@
 			)
 		)
-		(property "Footprint" "Components for Lamoka1 general:CAPC1005X55N"
+		(property "Footprint" "Capacitor_SMD:C_0402_1005Metric"
 			(at 79.7052 53.34 0)
 			(hide yes)
@@
 			)
 		)
-		(property "Footprint" "Components for Lamoka1 general:CAP_25SVPF100M"
+		(property "Footprint" "Capacitor_SMD:CP_Elec_8x11.9"
 			(at 136.8552 45.72 0)
 			(hide yes)
@@
 			)
 		)
-		(property "Footprint" ""
+		(property "Footprint" "Diode_SMD:D_SMA"
 			(at 113.03 85.09 0)
 			(hide yes)
@@
 			)
 		)
-		(property "Footprint" ""
+		(property "Footprint" "CSD16323Q3:DQG0008A"
 			(at 121.92 40.64 0)
 			(hide yes)
@@
 			)
 		)
-		(property "Footprint" "Components for Lamoka1 general:CAPC2012X140N"
+		(property "Footprint" "Capacitor_SMD:C_0805_2012Metric"
 			(at 109.22 84.1248 0)
 			(hide yes)
@@
 			)
 		)
-		(property "Footprint" "Components for Lamoka1 general:CAPC1005X55N"
+		(property "Footprint" "Capacitor_SMD:C_0402_1005Metric"
 			(at 72.0852 76.2 0)
 			(hide yes)
@@
 			)
 		)
-		(property "Footprint" ""
+		(property "Footprint" "Resistor_SMD:R_0201_0603Metric"
 			(at 142.24 83.058 90)
 			(hide yes)
@@
 			)
 		)
-		(property "Footprint" ""
+		(property "Footprint" "Resistor_SMD:R_0402_1005Metric"
 			(at 35.052 72.39 90)
 			(hide yes)
@@
 			)
 		)
-		(property "Footprint" ""
+		(property "Footprint" "Resistor_SMD:R_0402_1005Metric"
 			(at 62.992 41.91 90)
 			(hide yes)
@@
 			)
 		)
-		(property "Footprint" ""
+		(property "Footprint" "Resistor_SMD:R_0402_1005Metric"
 			(at 76.962 41.91 90)
 			(hide yes)
@@
 			)
 		)
-		(property "Footprint" ""
+		(property "Footprint" "Resistor_SMD:R_1206_3216Metric"
 			(at 92.71 39.878 90)
 			(hide yes)
@@
 			)
 		)
-		(property "Footprint" "Components for Lamoka1 general:CAP_25SVPF100M"
+		(property "Footprint" "Capacitor_SMD:CP_Elec_8x11.9"
 			(at 159.7152 45.72 0)
 			(hide yes)
@@
 			)
 		)
-		(property "Footprint" "Components for Lamoka1 general:IND_XAL1580-182MEB"
+		(property "Footprint" "Inductor_SMD:L_Coilcraft_XAL1580-182"
 			(at 107.95 38.1 0)
 			(hide yes)
@@
 			)
 		)
-		(property "Footprint" ""
+		(property "Footprint" "Resistor_SMD:R_0201_0603Metric"
 			(at 52.832 72.39 90)
 			(hide yes)
@@
 			)
 		)
-		(property "Footprint" "Components for Lamoka1 general:CAP_25SVPF100M"
+		(property "Footprint" "Capacitor_SMD:CP_Elec_8x11.9"
 			(at 148.2852 45.72 0)
 			(hide yes)
@@
 			)
 		)
-		(property "Footprint" ""
+		(property "Footprint" "Resistor_SMD:R_0402_1005Metric"
 			(at 127.762 50.8 90)
 			(hide yes)
