File: Lamoka1-DEV-Brain/Kicad files/Lamoka1-DEV-board.kicad_pcb (KiCad board)
At the start: 2 copper layers, 70 x 30 mm, 51 parts, among them J1 Conn_01x13_Pin, J3 USB_C_Receptacle_USB2.0_14P, SW1 PTS636 SM43J SMTR LFS, U1 RP2354A, U2 AMS1117-3.3, U3 74AHCT1G125, X1 ABM8-272-T3

Commit message: Cleaning up the DEV-Brains folder
Connections:
- net /GPOI1 renamed /GPIO1
- net /GPOI10 renamed /GPIO10
- net /GPOI2 renamed /GPIO2
- net /GPOI3 renamed /GPIO3
- net /GPOI4 renamed /GPIO4
- net /GPOI5 renamed /GPIO5
- net /GPOI6 renamed /GPIO6
- net /GPOI7 renamed /GPIO7
- net /GPOI9 renamed /GPIO9
