File: HARDWARE/kicadfiles/Lamoka1/Lamoka1/Inversion-section.kicad_sch (KiCad schematic)
At the start: 30 parts, among them Q1 NMOS, Q2 NMOS, Q3 NMOS, Q4 NMOS, Q5 NMOS, Q6 NMOS, U4 LM5122MH/NOPB

Commit message: Moving symbols and footprints into repo
Parts:
- Q3, Q4, Q5, Q6: value NMOS -> CSD19536KCS
Other:
- moved on the sheet: Q4, Q6
Changed lines of the file:
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@@
 			)
 		)
-		(property "Value" "NMOS"
+		(property "Value" "CSD19536KCS"
 			(at 256.54 64.7699 0)
 			(show_name no)
@@
 	(symbol
 		(lib_id "Simulation_SPICE:NMOS")
-		(at 284.48 63.5 180)
+		(at 293.37 63.5 180)
 		(unit 1)
 		(body_style 1)
@@
 		(fields_autoplaced yes)
 		(property "Reference" "Q4"
-			(at 278.13 62.2299 0)
+			(at 287.02 62.2299 0)
 			(show_name no)
 			(do_not_autoplace no)
@@
 			)
 		)
-		(property "Value" "NMOS"
-			(at 278.13 64.7699 0)
+		(property "Value" "CSD19536KCS"
+			(at 287.02 64.7699 0)
 			(show_name no)
 			(do_not_autoplace no)
@@
 		)
 		(property "Footprint" "Components for Lamoka1 general:TO254P1036X470X1965-3"
-			(at 279.4 66.04 0)
+			(at 288.29 66.04 0)
 			(hide yes)
 			(show_name no)
@@
 		)
 		(property "Datasheet" "https://ngspice.sourceforge.io/docs/ngspice-html-manual/manual.xhtml#cha_MOSFETs"
-			(at 284.48 50.8 0)
+			(at 293.37 50.8 0)
 			(hide yes)
 			(show_name no)
@@
 		)
 		(property "Description" "N-MOSFET transistor, drain/source/gate"
-			(at 284.48 63.5 0)
+			(at 293.37 63.5 0)
 			(hide yes)
 			(show_name no)
@@
 		)
 		(property "Sim.Device" "NMOS"
-			(at 284.48 46.355 0)
+			(at 293.37 46.355 0)
 			(hide yes)
 			(show_name no)
@@
 		)
 		(property "Sim.Type" "VDMOS"
-			(at 284.48 44.45 0)
+			(at 293.37 44.45 0)
 			(hide yes)
 			(show_name no)
@@
 		)
 		(property "Sim.Pins" "1=D 2=G 3=S"
-			(at 284.48 48.26 0)
+			(at 293.37 48.26 0)
 			(hide yes)
 			(show_name no)
@@
 			)
 		)
-		(property "Value" "NMOS"
+		(property "Value" "CSD19536KCS"
 			(at 256.54 83.8199 0)
 			(show_name no)
@@
 	(symbol
 		(lib_id "Simulation_SPICE:NMOS")
-		(at 284.48 81.28 180)
+		(at 293.37 81.28 180)
 		(unit 1)
 		(body_style 1)
@@
 		(fields_autoplaced yes)
 		(property "Reference" "Q6"
-			(at 278.13 80.0099 0)
+			(at 287.02 80.0099 0)
 			(show_name no)
 			(do_not_autoplace no)
@@
 			)
 		)
-		(property "Value" "NMOS"
-			(at 278.13 82.5499 0)
+		(property "Value" "CSD19536KCS"
+			(at 287.02 82.5499 0)
 			(show_name no)
 			(do_not_autoplace no)
@@
 		)
 		(property "Footprint" "Components for Lamoka1 general:TO254P1036X470X1965-3"
-			(at 279.4 83.82 0)
+			(at 288.29 83.82 0)
 			(hide yes)
 			(show_name no)
@@
 		)
 		(property "Datasheet" "https://ngspice.sourceforge.io/docs/ngspice-html-manual/manual.xhtml#cha_MOSFETs"
-			(at 284.48 68.58 0)
+			(at 293.37 68.58 0)
 			(hide yes)
 			(show_name no)
@@
 		)
 		(property "Description" "N-MOSFET transistor, drain/source/gate"
-			(at 284.48 81.28 0)
+			(at 293.37 81.28 0)
 			(hide yes)
 			(show_name no)
@@
 		)
 		(property "Sim.Device" "NMOS"
-			(at 284.48 64.135 0)
+			(at 293.37 64.135 0)
 			(hide yes)
 			(show_name no)
@@
 		)
 		(property "Sim.Type" "VDMOS"
-			(at 284.48 62.23 0)
+			(at 293.37 62.23 0)
 			(hide yes)
 			(show_name no)
@@
 		)
 		(property "Sim.Pins" "1=D 2=G 3=S"
-			(at 284.48 66.04 0)
-			(hide yes)
-			(show_name no)
+			(at 293.37 66.04 0)
+			(hide yes)
+			(show_name no)
