File: HARDWARE/Kicadfiles/Lamoka1/Inversion-section.kicad_sch (KiCad schematic)
At the start: 41 parts, among them Q1 25V 60A N-Ch, Q2 30V 56A N-Ch, Q3 100V 150A N-Ch, Q4 100V 150A N-Ch, Q5 100V 150A N-Ch, Q6 100V 150A N-Ch, U4 LM5122MH/NOPB, U5 UCC27735DR, U6 UCC27735DR, U9 TMP235A2DBZR

Commit message: Improving openSSF and Repograde rankings, Fixing misc PCB errors
Parts:
- U4: footprint LM5122QMHX-NOPB:PWP20_3P0X4P2 -> lm5122:PWP0020A_N
Changed lines of the file:
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@@
 			)
 		)
-		(property "Footprint" "LM5122QMHX-NOPB:PWP20_3P0X4P2"
+		(property "Footprint" "lm5122:PWP0020A_N"
 			(at 55.88 114.3 0)
 			(hide yes)
