File: HARDWARE/Kicadfiles/Lamoka1/Lamoka1.kicad_pcb (KiCad board)
At the start: 2 copper layers, 95 x 95 mm, 118 parts, among them IC1 INA240A2DR, J1 2606-1108/010-000, J2 2606-1352, J3 USB_C_Receptacle_USB2.0_14P, J4 FAN GND, J5 2604-1103, J6 FAN 5V, Q1 25V 60A N-Ch, Q2 30V 56A N-Ch, Q3 100V 150A N-Ch, Q4 100V 150A N-Ch, Q5 100V 150A N-Ch, Q6 100V 150A N-Ch, SW1 B3F-4055, U1 RP2354A, U10 ADS7128IRTER, U2 AMS1117-3.3, U3 74AHCT1G125, U4 LM5122MH/NOPB, U5 UCC27735DR, U6 UCC27735DR, U7 TPS62160DSGR, U8 TMP235A2DBZR, U9 TMP235A2DBZR, X1 ABM8-272-T3

Commit message: Routing H bridge paths, other various routing. Lamoka1/2
Parts:
- R10, R12, R17, R18: moved to B.Cu
- moved U9 31.1 mm to (221.3, 132.6), turned to 180 degrees
- moved C29 3.94 mm to (246.8, 130.1)
- moved R29 3.94 mm to (243.8, 129.3)
- moved R30 3.94 mm to (246.8, 128.5)
- moved R31 2.79 mm to (224.2, 128.6)
- moved C30 2.79 mm to (221.1, 127.8)
- moved R32 2.79 mm to (221.1, 129.3)
Routing:
- net /BLUE: track 203.0 -> 652.1 mm, vias 7 -> 28
- net /Inversion-Section/G4D: track 446.9 -> 854.0 mm, vias 9 -> 31
- net /BROWN: track 170.2 -> 351.6 mm, vias 6 -> 20
- net /Control-Section/GPIO1: track 0.00 -> 128.9 mm
- net /Control-Section/GPIO2: track 0.00 -> 127.7 mm
- net /Inversion-Section/CSP: track 328.0 -> 405.9 mm, vias 2 -> 5
- net /BLACK: track 59.8 -> 119.7 mm
- net /Control-Section/TEMP_INV: track 0.00 -> 45.6 mm, vias 0 -> 3
- net /RED: track 58.7 -> 101.8 mm
- net Net-(C20-Pad1): track 6.72 -> 30.4 mm
- net /Inversion-Section/HB1: track 6.90 -> 26.8 mm, vias 0 -> 1
- net /Control-Section/BTN: track 23.3 -> 41.8 mm, vias 0 -> 1
- net +BATT: track 41.6 -> 54.1 mm
- net /Control-Section/XIN: track 7.93 -> 20.3 mm
- net /Inversion-Section/HB2: track 14.4 -> 24.3 mm, vias 0 -> 1
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Other:
- board text added: "5V"
- board text added: "GND"

Commit message: finishing up routing and all of the lamoka1/2
Parts:
- moved Rfbt1 3.17 mm to (201.8, 168.4), turned to 180 degrees
Routing:
- net /Control-Section/3v3: track 65.2 -> 167.2 mm, vias 2 -> 11
- net /Control-Section/GPIO4: track 0.00 -> 64.1 mm, vias 0 -> 4
- net /Control-Section/GPIO3: track 0.00 -> 61.6 mm, vias 0 -> 4
- net /Control-Section/5V: track 109.7 -> 160.5 mm, vias 0 -> 1
- net /Inversion-Section/G4D: track 854.0 -> 884.4 mm, vias 31 -> 32
- net /Control-Section/1V1: track 12.9 -> 22.7 mm
- net GND: track 0.00 -> 9.03 mm, vias 30 -> 94
- net /Control-Section/GPIO2: track 127.7 -> 120.4 mm
- net /Control-Section/GPIO1: track 128.9 -> 121.7 mm
- net /BROWN: track 351.6 -> 344.7 mm
- net /Control-Section/AIN1: track 93.2 -> 87.8 mm
- net /Control-Section/TEMP_INV: track 45.6 -> 41.6 mm
- net /Control-Section/GPIO11: track 53.8 -> 52.3 mm, vias 1 -> 3
- net /Control-Section/AIN2: track 65.9 -> 67.0 mm
- net /Inversion-Section/FB: track 10.3 -> 11.4 mm
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- added copper zone on B.Cu, net /Control-Section/1V1
- added copper zone on F.Cu, net /Control-Section/1V1
- added copper zone on B.Cu, net /Control-Section/3v3
- added copper zone on F.Cu, net /Control-Section/3v3

Commit message: DRC fixes etc Lamoka1/2
Routing:
- net GND: track 9.03 -> 14.9 mm, vias 94 -> 156
- net /Control-Section/5V: track 160.5 -> 161.3 mm

Commit message: Improving openSSF and Repograde rankings, Fixing misc PCB errors
Parts:
- U4: footprint LM5122QMHX-NOPB:PWP20_3P0X4P2 -> lm5122:PWP0020A_N
- moved L2 82.5 mm to (154.3, 133.9)
- moved C15 82.5 mm to (127.0, 93.2)
- moved C21 82.5 mm to (142.8, 82.9)
- moved C23 82.5 mm to (169.3, 93.5)
- moved Ccomp2 82.5 mm to (138.2, 118.5)
- moved Cout1 82.5 mm to (187.7, 127.1)
- moved Cres1 82.5 mm to (144.7, 121.9)
- moved D1 82.5 mm to (128.9, 99.3)
- moved D2 82.5 mm to (136.1, 99.3)
- moved D3 82.5 mm to (143.3, 99.3)
- moved L3 82.5 mm to (108.3, 117.1)
- moved R19 82.5 mm to (101.8, 116.8)
- moved R23 82.5 mm to (157.3, 84.7)
- moved R31 82.5 mm to (161.0, 75.6)
- moved R33 82.5 mm to (126.5, 116.9)
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Routing:
- net GND: track 14.9 -> 32.6 mm, vias 156 -> 177
- net /Inversion-Section/COMP: track 8.52 -> 15.2 mm
- net /Inversion-Section/UVLO: track 21.3 -> 27.8 mm
- net /Inversion-Section/VIN: track 18.6 -> 24.9 mm, vias 1 -> 3
- net /BLUE: track 652.1 -> 646.1 mm, vias 28 -> 26
- net /Control-Section/GPIO3: track 61.6 -> 60.8 mm
- net /Control-Section/GPIO9: track 27.0 -> 27.8 mm
- net /Control-Section/GPIO4: track 64.1 -> 64.6 mm
