File: HARDWARE/Kicadfiles/Lamoka1-half/Control-section.kicad_sch (KiCad schematic)
At the start: 52 parts, among them IC1 INA240A2DR, U1 RP2354A, U10 ADS7128IRTER, U2 AMS1117-3.3, U7 TPS62160DSGR, U8 TMP235A2DBZR, X1 ABM8-272-T3

Commit message: Lamoka1/2: rename main board, regenerate fab/assembly package, add PIE V1.9
- Rename the main (non-DEV-Brain) board from Lamoka1 to Lamoka1/2 everywhere
  (paths, library nickname, gerbers, step, docs, BOM map).
- Regenerate the main-board fab/assembly submission package (gerbers, drill,
  PCBWay BOM + pick-and-place) from the current board; add tools/make_fab_bom.py.
- Add a reproducible board-image pipeline (tools/make_images.sh, `make images`)
  and refresh all six published images.
- Add PIE V1.9: first main-board firmware (5-LED UI ported from V1.8 plus the
  H-bridge power stage — explicit arming, PWM dead-time scheme verified by
  simulation, soft start, closed-loop regulation, supervisory protection,
  watchdog). Compiles clean.
- Update PIE-v1.9-information.md, SOFTWARE/README.md, Operation.md, AGENTS.md.
- Paid-model review pass applied; docs and tooling fixes (ruff, tests).
Parts:
- CR1, CR2: value 40V 1A Schottky -> SS14-E3/61T; footprint SS14-E3/61T:DO-214AC_VIS -> Lamoka1-half:DO-214AC_VIS
- L3: footprint PA4332.222NLT:IND_PA4332.222NLT_PUL -> Lamoka1-half:IND_PA4332.222NLT_PUL
- R24: footprint Resistor_SMD:R_0603_1608Metric -> Lamoka1-half:R_0603_1608Metric
- U2: footprint Package_TO_SOT_SMD:SOT-223-3_TabPin2 -> Lamoka1-half:SOT-223-3_TabPin2
- U7: footprint TPS62160DSGR:DSG8_1P6X0P9 -> Lamoka1-half:DSG8_1P6X0P9

Commit message: Fixes to meet claims
Parts:
- C13: value 10u -> 22uF; footprint Capacitor_SMD:C_0402_1005Metric -> Capacitor_Tantalum_SMD:CP_EIA-3216-18_Kemet-A; MPN CL05A106MQ5NUNC -> T491A226K010AT
- R27: value 43.2k -> 68k; MPN RC0603FR-0743K2L -> RC0603FR-0768KL
- R29, R31: value 45.3k -> 68k; MPN RC0603FR-0745K3L -> RC0603FR-0768KL
Changed lines of the file:
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@@
 			)
 		)
-		(property "Value" "45.3k"
+		(property "Value" "68k"
 			(at 90.17 199.3899 0)
 			(show_name no)
@@
 			)
 		)
-		(property "MPN" "RC0603FR-0745K3L"
+		(property "MPN" "RC0603FR-0768KL"
 			(at 87.63 198.12 0)
 			(hide yes)
@@
 			)
 		)
-		(property "Value" "10u"
+		(property "Value" "22uF"
 			(at 138.43 148.5899 0)
 			(show_name no)
@@
 			)
 		)
-		(property "Footprint" "Capacitor_SMD:C_0402_1005Metric"
+		(property "Footprint" "Capacitor_Tantalum_SMD:CP_EIA-3216-18_Kemet-A"
 			(at 135.5852 151.13 0)
 			(hide yes)
@@
 			)
 		)
-		(property "MPN" "CL05A106MQ5NUNC"
+		(property "MPN" "T491A226K010AT"
 			(at 134.62 147.32 0)
 			(hide yes)
@@
 			)
 		)
-		(property "Value" "43.2k"
+		(property "Value" "68k"
 			(at 62.23 198.1199 0)
 			(show_name no)
@@
 			)
 		)
-		(property "MPN" "RC0603FR-0743K2L"
+		(property "MPN" "RC0603FR-0768KL"
 			(at 59.69 196.85 0)
 			(hide yes)
@@
 			)
 		)
-		(property "Value" "45.3k"
+		(property "Value" "68k"
 			(at 118.11 199.3899 0)
 			(show_name no)
@@
 			)
 		)
-		(property "MPN" "RC0603FR-0745K3L"
+		(property "MPN" "RC0603FR-0768KL"
 			(at 115.57 198.12 0)
 			(hide yes)
