File: HARDWARE/Kicadfiles/Lamoka1-half/Inversion-section.kicad_sch (KiCad schematic)
At the start: 41 parts, among them Q1 25V 60A N-Ch, Q2 30V 56A N-Ch, Q3 100V 150A N-Ch, Q4 100V 150A N-Ch, Q5 100V 150A N-Ch, Q6 100V 150A N-Ch, U4 LM5122MH/NOPB, U5 UCC27735DR, U6 UCC27735DR, U9 TMP235A2DBZR

Commit message: Lamoka1/2: rename main board, regenerate fab/assembly package, add PIE V1.9
- Rename the main (non-DEV-Brain) board from Lamoka1 to Lamoka1/2 everywhere
  (paths, library nickname, gerbers, step, docs, BOM map).
- Regenerate the main-board fab/assembly submission package (gerbers, drill,
  PCBWay BOM + pick-and-place) from the current board; add tools/make_fab_bom.py.
- Add a reproducible board-image pipeline (tools/make_images.sh, `make images`)
  and refresh all six published images.
- Add PIE V1.9: first main-board firmware (5-LED UI ported from V1.8 plus the
  H-bridge power stage — explicit arming, PWM dead-time scheme verified by
  simulation, soft start, closed-loop regulation, supervisory protection,
  watchdog). Compiles clean.
- Update PIE-v1.9-information.md, SOFTWARE/README.md, Operation.md, AGENTS.md.
- Paid-model review pass applied; docs and tooling fixes (ruff, tests).
Parts:
- Cout1: footprint Capacitor_SMD:CP_Elec_8x11.9 -> Lamoka1-half:CP_Elec_8x11.9_Cout1
- Cout2: footprint Capacitor_SMD:CP_Elec_8x11.9 -> Lamoka1-half:CP_Elec_8x11.9_Cout2
- Cout3: footprint Capacitor_SMD:CP_Elec_8x11.9 -> Lamoka1-half:CP_Elec_8x11.9_Cout3
- D11, D12: value D -> SS14-E3/61T
- D6: value D -> SK215ATR
- Q1: footprint CSD16323Q3:DQG0008A -> Lamoka1-half:DQG0008A
- Q2: footprint CSD17304Q3:DQG0008A -> Lamoka1-half:DQG0008A
- Q3, Q4, Q5, Q6: symbol Lamoka1_MOSFET:CSD19536KCS -> Lamoka1-half_MOSFET:CSD19536KCS
- U4: value LM5122MH/NOPB -> LM5122MHX/NOPB; footprint lm5122:PWP0020A_N -> Lamoka1-half:PWP0020A_N; MPN LM5122MH/NOPB -> LM5122MHX/NOPB

Commit message: Fixes to meet claims
Parts:
- added C34, C36: 10uF, Capacitor_SMD:C_0805_2012Metric, symbol Device:C
- added C35, C37: 100nF, Capacitor_SMD:C_0603_1608Metric, symbol Device:C
- Ccomp1: value 3.9nF -> 15nF; MPN CGA4C2C0G1H392J060AA -> CGA4F1C0G2A153J085AE
- Ccomp2: value 130pF -> 44.8pF; MPN GRM1555C1H131GA01D -> GRM1555C1H448JA01D
- Cout1, Cout2, Cout3: MPN 25SVPF180M -> 35SVPK180M
- Coutx1: value 47uF -> 22uF; MPN C3216X5R1E476M160AC -> C3216X5R1V226M160AC
- Q1: value 25V 60A N-Ch -> 30V 56A N-Ch; MPN CSD16323Q3 -> CSD17304Q3
- Rcomp1: value 28.7k -> 80.6k; MPN RC0201FR-0728K7L -> RC0201FR-0780K6L
- Rfbt1: value 49.9k -> 64.9k; MPN CRCW040249K9FKED -> CRCW040264K9FKED
- Rsense1: footprint Resistor_SMD:R_1206_3216Metric -> Resistor_SMD:R_2512_6332Metric; MPN CSNL1206FT2L00 -> CSNL2512FT2L00; Manufacturer (none) -> Stackpole
- Rslope1: value 105k -> 49.9k; MPN RC0201FR-07105KL -> RC0201FR-0749K9L
Connections:
- net CSP: now also C34.2, C35.2, C36.2, C37.2
- net GND: now also C34.1, C35.1, C36.1, C37.1
