File: HARDWARE/Kicadfiles/Lamoka1-half/Lamoka1-half.kicad_pcb (KiCad board)
At the start: 2 copper layers, 95 x 95 mm, 118 parts, among them IC1 INA240A2DR, J1 2606-1108/010-000, J2 2606-1352, J3 USB_C_Receptacle_USB2.0_14P, J4 FAN GND, J5 2604-1103, J6 FAN 5V, Q1 25V 60A N-Ch, Q2 30V 56A N-Ch, Q3 100V 150A N-Ch, Q4 100V 150A N-Ch, Q5 100V 150A N-Ch, Q6 100V 150A N-Ch, SW1 B3F-4055, U1 RP2354A, U10 ADS7128IRTER, U2 AMS1117-3.3, U3 74AHCT1G125, U4 LM5122MH/NOPB, U5 UCC27735DR, U6 UCC27735DR, U7 TPS62160DSGR, U8 TMP235A2DBZR, U9 TMP235A2DBZR, X1 ABM8-272-T3

Commit message: Lamoka1/2: rename main board, regenerate fab/assembly package, add PIE V1.9
- Rename the main (non-DEV-Brain) board from Lamoka1 to Lamoka1/2 everywhere
  (paths, library nickname, gerbers, step, docs, BOM map).
- Regenerate the main-board fab/assembly submission package (gerbers, drill,
  PCBWay BOM + pick-and-place) from the current board; add tools/make_fab_bom.py.
- Add a reproducible board-image pipeline (tools/make_images.sh, `make images`)
  and refresh all six published images.
- Add PIE V1.9: first main-board firmware (5-LED UI ported from V1.8 plus the
  H-bridge power stage — explicit arming, PWM dead-time scheme verified by
  simulation, soft start, closed-loop regulation, supervisory protection,
  watchdog). Compiles clean.
- Update PIE-v1.9-information.md, SOFTWARE/README.md, Operation.md, AGENTS.md.
- Paid-model review pass applied; docs and tooling fixes (ruff, tests).
Parts:
- CR1, CR2: value 40V 1A Schottky -> SS14-E3/61T; footprint SS14-E3/61T:DO-214AC_VIS -> Lamoka1-half:DO-214AC_VIS
- Cout1: footprint Capacitor_SMD:CP_Elec_8x11.9 -> Lamoka1-half:CP_Elec_8x11.9_Cout1
- Cout2: footprint Capacitor_SMD:CP_Elec_8x11.9 -> Lamoka1-half:CP_Elec_8x11.9_Cout2
- Cout3: footprint Capacitor_SMD:CP_Elec_8x11.9 -> Lamoka1-half:CP_Elec_8x11.9_Cout3
- D11, D12: value D -> SS14-E3/61T
- D6: value D -> SK215ATR
- J1: footprint 2606-1108/010-000:CONN8_2606-1108&slash_010-000_WAG -> Lamoka1-half:CONN8_2606-1108&slash_010-000_WAG
- J2: footprint 2606-1352:CONN2_2606-1352_WAG -> Lamoka1-half:CONN2_2606-1352_WAG
- J5: footprint 2604-1103:CONN3_2604-1103_WAG -> Lamoka1-half:CONN3_2604-1103_WAG
- L3: footprint PA4332.222NLT:IND_PA4332.222NLT_PUL -> Lamoka1-half:IND_PA4332.222NLT_PUL
- Q1: footprint CSD16323Q3:DQG0008A -> Lamoka1-half:DQG0008A
- Q2: footprint CSD17304Q3:DQG0008A -> Lamoka1-half:DQG0008A
- R24: footprint Resistor_SMD:R_0603_1608Metric -> Lamoka1-half:R_0603_1608Metric
- U2: footprint Package_TO_SOT_SMD:SOT-223-3_TabPin2 -> Lamoka1-half:SOT-223-3_TabPin2
- U4: value LM5122MH/NOPB -> LM5122MHX/NOPB; footprint lm5122:PWP0020A_N -> Lamoka1-half:PWP0020A_N
- U7: footprint TPS62160DSGR:DSG8_1P6X0P9 -> Lamoka1-half:DSG8_1P6X0P9
Routing:
- net /BLACK: track 119.7 -> 118.0 mm

Commit message: Fixes to meet claims
Parts:
- added C34: 10uF, Capacitor_SMD:C_0805_2012Metric, B.Cu at (181.8, 119.5)
- added C35: 100nF, Capacitor_SMD:C_0603_1608Metric, B.Cu at (183.9, 119.5)
- added C36: 10uF, Capacitor_SMD:C_0805_2012Metric, B.Cu at (186.6, 86.0)
- added C37: 100nF, Capacitor_SMD:C_0603_1608Metric, B.Cu at (188.4, 86.0)
- C13: value 10u -> 22uF; footprint Capacitor_SMD:C_0402_1005Metric -> Capacitor_Tantalum_SMD:CP_EIA-3216-18_Kemet-A
- Ccomp1: value 3.9nF -> 15nF
- Ccomp2: value 130pF -> 44.8pF
- Coutx1: value 47uF -> 22uF
- Q1: value 25V 60A N-Ch -> 30V 56A N-Ch
- R27: value 43.2k -> 68k
- R29, R31: value 45.3k -> 68k
- Rcomp1: value 28.7k -> 80.6k
- Rfbt1: value 49.9k -> 64.9k
- Rsense1: footprint Resistor_SMD:R_1206_3216Metric -> Resistor_SMD:R_2512_6332Metric
- Rslope1: value 105k -> 49.9k
- moved C13 6.07 mm to (119.0, 117.6)
- moved Rsense1 4.12 mm to (142.2, 130.1)
Connections:
- J5 pad 3: GND -> /PE
- J5 pad 4: GND -> /PE
Routing:
- net /PE: track 0.00 -> 8.20 mm
- net /Inversion-Section/CSN: track 54.6 -> 58.0 mm
- net /Inversion-Section/CSP: track 405.9 -> 409.0 mm
- net /Control-Section/3v3: track 167.0 -> 169.6 mm
