File: HARDWARE/Kicadfiles/Lamoka1-half/Lamoka1-half.kicad_sch (KiCad schematic)
At the start: 9 parts, among them J1 2606-1108/010-000, J2 2606-1352, J3 USB_C_Receptacle_USB2.0_14P, J4 FAN GND, J5 2604-1103, J6 FAN 5V

Commit message: Lamoka1/2: rename main board, regenerate fab/assembly package, add PIE V1.9
- Rename the main (non-DEV-Brain) board from Lamoka1 to Lamoka1/2 everywhere
  (paths, library nickname, gerbers, step, docs, BOM map).
- Regenerate the main-board fab/assembly submission package (gerbers, drill,
  PCBWay BOM + pick-and-place) from the current board; add tools/make_fab_bom.py.
- Add a reproducible board-image pipeline (tools/make_images.sh, `make images`)
  and refresh all six published images.
- Add PIE V1.9: first main-board firmware (5-LED UI ported from V1.8 plus the
  H-bridge power stage — explicit arming, PWM dead-time scheme verified by
  simulation, soft start, closed-loop regulation, supervisory protection,
  watchdog). Compiles clean.
- Update PIE-v1.9-information.md, SOFTWARE/README.md, Operation.md, AGENTS.md.
- Paid-model review pass applied; docs and tooling fixes (ruff, tests).
Parts:
- J1: footprint 2606-1108/010-000:CONN8_2606-1108&slash_010-000_WAG -> Lamoka1-half:CONN8_2606-1108&slash_010-000_WAG; MPN (none) -> 2606-1108/010-000
- J2: footprint 2606-1352:CONN2_2606-1352_WAG -> Lamoka1-half:CONN2_2606-1352_WAG; MPN (none) -> 2606-1352
- J4, J6: now left out of the parts list
- J5: footprint 2604-1103:CONN3_2604-1103_WAG -> Lamoka1-half:CONN3_2604-1103_WAG; MPN (none) -> 2604-1103
Connections:
- net Control-Section/GND is gone; now on net Control-Section/GND: J3.SH (SHIELD)
Changed lines of the file:
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@@
 		)
 		(instances
-			(project "Lamoka1"
+			(project "Lamoka1-half"
 				(path "/c7bb62b6-932f-49c1-a356-0286e905fc0a"
 					(reference "H1")
@@
 			)
 		)
-		(property "Footprint" "2606-1352:CONN2_2606-1352_WAG"
+		(property "Footprint" "Lamoka1-half:CONN2_2606-1352_WAG"
 			(at 151.13 24.13 0)
 			(hide yes)
@@
 			)
 		)
+		(property "MPN" "2606-1352"
+			(at 151.13 24.13 0)
+			(hide yes)
+			(show_name no)
+			(do_not_autoplace no)
+			(effects
+				(font
+					(size 1.27 1.27)
+				)
+			)
+		)
 		(property "Description" ""
 			(at 151.13 24.13 0)
@@
 		)
 		(instances
-			(project "Lamoka1"
+			(project "Lamoka1-half"
 				(path "/c7bb62b6-932f-49c1-a356-0286e905fc0a"
 					(reference "J2")
@@
 			)
 		)
-		(property "Footprint" "2604-1103:CONN3_2604-1103_WAG"
+		(property "Footprint" "Lamoka1-half:CONN3_2604-1103_WAG"
 			(at 260.35 72.39 0)
 			(hide yes)
@@
 			)
 		)
+		(property "MPN" "2604-1103"
+			(at 260.35 72.39 0)
+			(hide yes)
+			(show_name no)
+			(do_not_autoplace no)
+			(effects
+				(font
+					(size 1.27 1.27)
+				)
+			)
+		)
 		(property "Description" ""
 			(at 260.35 72.39 0)
@@
 		)
 		(instances
-			(project "Lamoka1"
+			(project "Lamoka1-half"
 				(path "/c7bb62b6-932f-49c1-a356-0286e905fc0a"
 					(reference "J5")
@@
 			)
 		)
-		(property "Footprint" "2606-1108/010-000:CONN8_2606-1108&slash_010-000_WAG"
+		(property "Footprint" "Lamoka1-half:CONN8_2606-1108&slash_010-000_WAG"
 			(at 227.33 35.56 0)
 			(hide yes)
@@
 			)
 		)
+		(property "MPN" "2606-1108/010-000"
+			(at 227.33 35.56 0)
+			(hide yes)
+			(show_name no)
+			(do_not_autoplace no)
+			(effects
+				(font
+					(size 1.27 1.27)
+				)
+			)
+		)
 		(property "Description" ""
 			(at 227.33 35.56 0)
@@
 		)
 		(instances
-			(project "Lamoka1"
+			(project "Lamoka1-half"
 				(path "/c7bb62b6-932f-49c1-a356-0286e905fc0a"
 					(reference "J1")
@@
 		)
 		(instances
-			(project "Lamoka1"
+			(project "Lamoka1-half"
 				(path "/c7bb62b6-932f-49c1-a356-0286e905fc0a"
 					(reference "#G1")
@@
 		)
 		(instances
-			(project "Lamoka1"
+			(project "Lamoka1-half"
 				(path "/c7bb62b6-932f-49c1-a356-0286e905fc0a"
 					(reference "H2")
@@
 		(body_style 1)
 		(exclude_from_sim no)
-		(in_bom yes)
+		(in_bom no)
 		(on_board yes)
 		(in_pos_files yes)
@@
 		)
 		(instances
-			(project "Lamoka1"
+			(project "Lamoka1-half"
 				(path "/c7bb62b6-932f-49c1-a356-0286e905fc0a"
 					(reference "J4")
@@
 		)
 		(instances
-			(project "Lamoka1"
+			(project "Lamoka1-half"
 				(path "/c7bb62b6-932f-49c1-a356-0286e905fc0a"
 					(reference "J3")
@@
 		)
 		(instances
-			(project "Lamoka1"
+			(project "Lamoka1-half"
 				(path "/c7bb62b6-932f-49c1-a356-0286e905fc0a"
 					(reference "RCS1")
@@
 		)
 		(instances
-			(project "Lamoka1"
+			(project "Lamoka1-half"
 				(path "/c7bb62b6-932f-49c1-a356-0286e905fc0a"
 					(reference "#PWR046")
@@
 		(body_style 1)
 		(exclude_from_sim no)
-		(in_bom yes)
+		(in_bom no)
 		(on_board yes)
 		(in_pos_files yes)
@@
 		)
 		(instances
-			(project "Lamoka1"
+			(project "Lamoka1-half"
 				(path "/c7bb62b6-932f-49c1-a356-0286e905fc0a"
 					(reference "J6")
@@
 		)
 		(instances
-			(project "Lamoka1"
+			(project "Lamoka1-half"
 				(path "/c7bb62b6-932f-49c1-a356-0286e905fc0a"
 					(reference "#FLG01")
@@
 		)
 		(instances
-			(project "Lamoka1"
+			(project "Lamoka1-half"
 				(path "/c7bb62b6-932f-49c1-a356-0286e905fc0a"
 					(page "3")
@@
 		)
 		(instances
-			(project "Lamoka1"
+			(project "Lamoka1-half"
 				(path "/c7bb62b6-932f-49c1-a356-0286e905fc0a"
 					(page "2")
@@
 		)
 		(instances
-			(project "Lamoka1"
+			(project "Lamoka1-half"
 				(path "/c7bb62b6-932f-49c1-a356-0286e905fc0a"
 					(page "4")

Commit message: Improvements to general Lamoka1/2
Connections:
- net Control-Section/GND is gone; now on net Control-Section/GND: J3.SH (SHIELD)
Changed lines of the file:
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@@
+			)
+		)
+		(property "Description" ""
+			(at 151.13 24.13 0)
+			(hide yes)
+			(show_name no)
+			(do_not_autoplace no)
+			(effects
+				(font
+					(size 1.27 1.27)
+				)
 			)
 		)
 		(property "MPN" "2606-1352"
-			(at 151.13 24.13 0)
-			(hide yes)
-			(show_name no)
-			(do_not_autoplace no)
-			(effects
-				(font
-					(size 1.27 1.27)
-				)
-			)
-		)
-		(property "Description" ""
 			(at 151.13 24.13 0)
 			(hide yes)
@@
 			)
 		)
+		(property "Description" ""
+			(at 260.35 72.39 0)
+			(hide yes)
+			(show_name no)
+			(do_not_autoplace no)
+			(effects
+				(font
+					(size 1.27 1.27)
+				)
+			)
+		)
 		(property "MPN" "2604-1103"
-			(at 260.35 72.39 0)
-			(hide yes)
-			(show_name no)
-			(do_not_autoplace no)
-			(effects
-				(font
-					(size 1.27 1.27)
-				)
-			)
-		)
-		(property "Description" ""
 			(at 260.35 72.39 0)
 			(hide yes)
@@
 			)
 		)
+		(property "Description" ""
+			(at 227.33 35.56 0)
+			(hide yes)
+			(show_name no)
+			(do_not_autoplace no)
+			(effects
+				(font
+					(size 1.27 1.27)
+				)
+			)
+		)
 		(property "MPN" "2606-1108/010-000"
 			(at 227.33 35.56 0)
 			(hide yes)
-			(show_name no)
-			(do_not_autoplace no)
-			(effects
-				(font
-					(size 1.27 1.27)
-				)
-			)
-		)
-		(property "Description" ""
-			(at 227.33 35.56 0)
-			(hide yes)

Commit message: Fixes to meet claims
Connections:
- net Control-Section/GND is gone; now on net Control-Section/GND: J3.SH (SHIELD)
- net GND: no longer J5.3 (2_1), J5.4 (2_2)
- new net PE: J5.3 (2_1), J5.4 (2_2)
Changed lines of the file:
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@@
-	)
-	(junction
-		(at 254 78.74)
-		(diameter 0)
-		(color 0 0 0 0)
 	)
 	(junction
@@
 	(wire
 		(pts
-			(xy 254 77.47) (xy 254 78.74)
-		)
-		(stroke
-			(width 0)
-			(type default)
-		)
-	)
-	(wire
-		(pts
 			(xy 20.32 114.3) (xy 20.32 111.76)
 		)
@@
 	(wire
 		(pts
+			(xy 229.87 78.74) (xy 232.41 78.74)
+		)
+		(stroke
+			(width 0)
+			(type default)
+		)
+	)
+	(wire
+		(pts
 			(xy 144.78 30.48) (xy 149.86 30.48)
 		)
@@
 	(wire
 		(pts
-			(xy 254 78.74) (xy 254 80.01)
+			(xy 254 77.47) (xy 254 80.01)
 		)
 		(stroke
@@
 		(pts
 			(xy 49.53 92.71) (xy 63.5 92.71)
-		)
-		(stroke
-			(width 0)
-			(type default)
-		)
-	)
-	(wire
-		(pts
-			(xy 229.87 78.74) (xy 254 78.74)
 		)
 		(stroke
@@
 		)
 	)
-	(label "GND"
+	(label "PE"
 		(at 260.35 77.47 180)
 		(effects
@@
 		)
 	)
+	(label "GND"
+		(at 232.41 78.74 0)
+		(effects
+			(font
+				(size 1.27 1.27)
+			)
+			(justify left bottom)
+		)
+	)
